File: demos/5v_rail_power/docs/FiveVoltRailPower.kicad_sch (KiCad schematic)
At the start: 7 parts, among them P1 Header1xNMale, U1 L7805

Commit message: export: kicad_sch — Phase 2.5b: layered placement + routing + KiCad 9 fix
Placement (placement.py, complete rewrite):
- Replaces naive grid with Layered Signal Flow algorithm (spec §5 stages 1–8)
- Stage 1: band classification — power chips/rails at top, LEDs at bottom,
  everything else in the signal band
- Stage 2: signal-flow DAG via BFS from Rail/Connector sources; layer = BFS
  distance from nearest source
- Stage 3–4: place within (band, layer) cells at 1500-mil (38.1 mm) same-band
  spacing, 1000-mil inter-band gutter, 25.4 mm page margin
- Stage 6: cluster breakup — up to 10 iterations shifting same-band parts
  that land closer than 0.9× SAME_BAND_SPACING_MM
- Stage 8: page sized to fit (A4 → A3 → A2 → A1)
- grid_place() and sheet_size_mm() kept as shims for backward-compat

Routing (routing.py, new file):
- route_net(): connects stub ends with Manhattan L-shapes (horizontal first)
- find_junctions(): returns points where ≥3 wire endpoints coincide
- renderer uses routed wires between signal-net stub ends

Hierarchical (hierarchical.py, new file):
- collect_boards(), is_multi_board(), sub_sheet_filename() — interface stub
  for multi-Board sub-sheet emission (full implementation deferred)

KiCad 9 sub-symbol name fix (library_loader.py):
- KiCad 9 schematics expect sub-symbols nested inside their parent in
  lib_symbols to use the bare name (R_0_1, LED_0_1, 4069_1_0) — NOT the
  lib-qualified name (Device:R_0_1, Device:LED_0_1, 4xxx:4069_1_0)
- Fixed _qualify_names() to add the lib: prefix only to the exact parent
  symbol name using a lookahead (?=") that prevents sub-unit names from
  being qualified

Tests (+25 tests):
- test_placement.py: band classification, all-on-grid, determinism,
  minimum spacing, power < signal < indicator Y ordering, page sizing
- test_routing.py: H/V segments, L-shapes, orthogonality, grid snap,
  junction detection

Golden files regenerated for all 23 demo designs.
Connections:
- net Net-(C1-t1) is gone; now on net Net-(BT1-neg): C1.2, U1.1 (IN)
- net Net-(D3-anode) is gone; now on net Net-(C2-t1): D3.1 (K), R1.1
Other:
- moved on the sheet: C1, C2, D1, D3, P1, R1, U1
