File: demos/doorbell_protector/docs/DoorbellProtector.kicad_sch (KiCad schematic)
At the start: 15 parts

Commit message: units: Ohms.__str__ uses engineering notation (kΩ, MΩ, GΩ) (#33)
* units: Ohms.__str__ uses engineering notation (kΩ, MΩ, GΩ)

The previous `Ohms.__str__` formatted with bare `:.3g`, producing
unreadable scientific output for clean kilo / mega multiples:

  str(Ohms(10_000))     == "1e+04 Ω"      → now "10 kΩ"
  str(Ohms(100_000))    == "1e+05 Ω"      → now "100 kΩ"
  str(Ohms(1_000_000))  == "1e+06 Ω"      → now "1 MΩ"

The breadboard SVG visualiser surfaced the problem: a resistor body
labelled "100000Ω" makes a reader count zeros, while a label of
"100 kΩ" reads at a glance — exactly the convention every schematic
and parts catalogue uses. Centralising the engineering notation in
`Ohms.__str__` means every downstream consumer (assembly guide,
breadboard SVG, kicad netlist, BOM, reports) inherits the readable
form without each format adapter rolling its own formatter.

  - `Ohms.__str__` returns "47 Ω", "4.7 kΩ", "10 kΩ", "100 kΩ",
    "1 MΩ", "10 MΩ", "1 GΩ" per the kilo / mega / giga thresholds.
  - `Resistor.__str__` delegates to `str(self._ohms)` so it
    inherits the new notation (was producing the noisy "47.0 Ω"
    via raw float).
  - The breadboard visualiser's resistor body label uses
    `str(part.ohms)` directly (previously had a private
    `_format_ohms_compact` helper; removed).
  - `tests/components/test_resistor.py::test_str` updated for
    "47 Ω" (was "47.0 Ω"); new `test_str_renders_in_engineering_notation`
    pins kΩ / MΩ output across the kilo and mega thresholds.
  - All demo docs / goldens refreshed where the Ohms.__str__
    change affected the rendered output (breadboard SVGs, kicad
    sch value fields, BOM rows).

* units: Farads + Henries __str__ also use engineering notation

Same treatment as `Ohms.__str__` (previous commit) for the other two
passive engineering quantities. Demos contain caps and inductors
with values that the bare `:.3g` formatter would emit in scientific
form (`1e-07 F` for a 100 nF decoupling cap); centralising t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
Parts:
- C1, C3, C4: value 1e-07 F -> 100 nF
- C2: value 4.7e-06 F -> 4.7 µF
- C5: value 4.7e-05 F -> 47 µF
- R1, R4: value 1e+03 Ω -> 1 kΩ
- R2, R3, R6: value 1e+06 Ω -> 1 MΩ
- R5: value 1e+04 Ω -> 10 kΩ
- R7: value 4.7e+03 Ω -> 4.7 kΩ
- R8: value 4.7e+04 Ω -> 47 kΩ
Changed lines of the file:
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@@
       (effects (font (size 1.27 1.27)))
     )
-    (property "Value" "1e+03 Ω"
+    (property "Value" "1 kΩ"
       (at 63.5 485.14 0)
       (effects (font (size 1.27 1.27)))
@@
       (effects (font (size 1.27 1.27)))
     )
-    (property "Value" "1e+06 Ω"
+    (property "Value" "1 MΩ"
       (at 63.5 523.24 0)
       (effects (font (size 1.27 1.27)))
@@
       (effects (font (size 1.27 1.27)))
     )
-    (property "Value" "1e+06 Ω"
+    (property "Value" "1 MΩ"
       (at 63.5 561.34 0)
       (effects (font (size 1.27 1.27)))
@@
       (effects (font (size 1.27 1.27)))
     )
-    (property "Value" "1e+03 Ω"
+    (property "Value" "1 kΩ"
       (at 63.5 599.44 0)
       (effects (font (size 1.27 1.27)))
@@
       (effects (font (size 1.27 1.27)))
     )
-    (property "Value" "1e+04 Ω"
+    (property "Value" "10 kΩ"
       (at 63.5 637.54 0)
       (effects (font (size 1.27 1.27)))
@@
       (effects (font (size 1.27 1.27)))
     )
-    (property "Value" "1e+06 Ω"
+    (property "Value" "1 MΩ"
       (at 63.5 675.64 0)
       (effects (font (size 1.27 1.27)))
@@
       (effects (font (size 1.27 1.27)))
     )
-    (property "Value" "4.7e+03 Ω"
+    (property "Value" "4.7 kΩ"
       (at 63.5 713.74 0)
       (effects (font (size 1.27 1.27)))
@@
       (effects (font (size 1.27 1.27)))
     )
-    (property "Value" "4.7e+04 Ω"
+    (property "Value" "47 kΩ"
       (at 63.5 751.84 0)
       (effects (font (size 1.27 1.27)))
@@
       (effects (font (size 1.27 1.27)))
     )
-    (property "Value" "1e-07 F"
+    (property "Value" "100 nF"
       (at 63.5 27.94 0)
       (effects (font (size 1.27 1.27)))
@@
       (effects (font (size 1.27 1.27)))
     )
-    (property "Value" "4.7e-06 F"
+    (property "Value" "4.7 µF"
       (at 63.5 66.04 0)
       (effects (font (size 1.27 1.27)))
@@
       (effects (font (size 1.27 1.27)))
     )
-    (property "Value" "1e-07 F"
+    (property "Value" "100 nF"
       (at 63.5 104.14 0)
       (effects (font (size 1.27 1.27)))
@@
       (effects (font (size 1.27 1.27)))
     )
-    (property "Value" "1e-07 F"
+    (property "Value" "100 nF"
       (at 63.5 142.24 0)
       (effects (font (size 1.27 1.27)))
@@
       (effects (font (size 1.27 1.27)))
     )
-    (property "Value" "4.7e-05 F"
+    (property "Value" "47 µF"
       (at 63.5 180.34 0)
       (effects (font (size 1.27 1.27)))
