File: demos/fan_cooling/docs/CooledSystem.kicad_sch (KiCad schematic)
At the start: 8 parts, among them J1 Header1xNFemale, J2 Header1xNFemale, P1 Header1xNMale, U2 SN74AHC1G14

Commit message: export: kicad_sch — Phase 2.5b: layered placement, wire routing, KiCad 10 compatibility (#23)
* export: kicad_sch — Phase 2.5b: layered placement + routing + KiCad 9 fix

Placement (placement.py, complete rewrite):
- Replaces naive grid with Layered Signal Flow algorithm (spec §5 stages 1–8)
- Stage 1: band classification — power chips/rails at top, LEDs at bottom,
  everything else in the signal band
- Stage 2: signal-flow DAG via BFS from Rail/Connector sources; layer = BFS
  distance from nearest source
- Stage 3–4: place within (band, layer) cells at 1500-mil (38.1 mm) same-band
  spacing, 1000-mil inter-band gutter, 25.4 mm page margin
- Stage 6: cluster breakup — up to 10 iterations shifting same-band parts
  that land closer than 0.9× SAME_BAND_SPACING_MM
- Stage 8: page sized to fit (A4 → A3 → A2 → A1)
- grid_place() and sheet_size_mm() kept as shims for backward-compat

Routing (routing.py, new file):
- route_net(): connects stub ends with Manhattan L-shapes (horizontal first)
- find_junctions(): returns points where ≥3 wire endpoints coincide
- renderer uses routed wires between signal-net stub ends

Hierarchical (hierarchical.py, new file):
- collect_boards(), is_multi_board(), sub_sheet_filename() — interface stub
  for multi-Board sub-sheet emission (full implementation deferred)

KiCad 9 sub-symbol name fix (library_loader.py):
- KiCad 9 schematics expect sub-symbols nested inside their parent in
  lib_symbols to use the bare name (R_0_1, LED_0_1, 4069_1_0) — NOT the
  lib-qualified name (Device:R_0_1, Device:LED_0_1, 4xxx:4069_1_0)
- Fixed _qualify_names() to add the lib: prefix only to the exact parent
  symbol name using a lookahead (?=") that prevents sub-unit names from
  being qualified

Tests (+25 tests):
- test_placement.py: band classification, all-on-grid, determinism,
  minimum spacing, power < signal < indicator Y ordering, page sizing
- test_routing.py: H/V segments, L-shapes, orthogonality, grid snap,
  junction detection

Golden files re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
Other:
- moved on the sheet: D1, J1, J2, P1, R1, R2, R3
Changed lines of the file:
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@@
 (kicad_sch
-  (version 20240618)
+  (version 20250114)
   (generator "wirebench")
-  (generator_version "0.1")
-  (paper "A3")
+  (generator_version "0.2")
+  (paper "A2")
   (symbol
     (lib_id "Connector_Generic:Conn_01x04")
-    (at 30.48 30.48 0)
+    (at 25.4 101.6 0)
     (unit 1)
     (exclude_from_sim no)
@@
     (dnp no)
     (property "Reference" "P1"
-      (at 33.02 27.94 0)
+      (at 27.94 99.06 0)
       (effects (font (size 1.27 1.27)))
     )
     (property "Value" "Header1xNMale"
-      (at 30.48 33.02 0)
+      (at 25.4 104.14 0)
       (effects (font (size 1.27 1.27)))
     )
@@
   )
   (wire
-    (pts (xy 25.4 33.02) (xy 22.86 33.02))
+    (pts (xy 20.32 104.14) (xy 17.78 104.14))
     (stroke (width 0) (type default))
   )
   (symbol
     (lib_id "power:VCC")
-    (at 22.86 33.02 90)
+    (at 17.78 104.14 90)
     (unit 1)
     (exclude_from_sim no)
@@
     (dnp no)
     (property "Reference" "#PWR"
-      (at 22.86 33.02 0)
+      (at 17.78 104.14 0)
       (effects (font (size 1.27 1.27)) (hide yes))
     )
     (property "Value" "VCC"
-      (at 22.86 33.02 0)
-      (effects (font (size 1.27 1.27)))
-    )
-    (pin "1")
-  )
-  (wire
-    (pts (xy 25.4 30.48) (xy 22.86 30.48))
+      (at 17.78 104.14 0)
+      (effects (font (size 1.27 1.27)))
+    )
+    (pin "1")
+  )
+  (wire
+    (pts (xy 20.32 101.6) (xy 17.78 101.6))
     (stroke (width 0) (type default))
   )
   (symbol
     (lib_id "power:GND")
-    (at 22.86 30.48 270)
+    (at 17.78 101.6 270)
     (unit 1)
     (exclude_from_sim no)
@@
     (dnp no)
     (property "Reference" "#PWR"
-      (at 22.86 30.48 0)
+      (at 17.78 101.6 0)
       (effects (font (size 1.27 1.27)) (hide yes))
     )
     (property "Value" "GND"
-      (at 22.86 30.48 0)
-      (effects (font (size 1.27 1.27)))
-    )
-    (pin "1")
-  )
-  (wire
-    (pts (xy 25.4 27.94) (xy 22.86 27.94))
-    (stroke (width 0) (type default))
-  )
-  (wire
-    (pts (xy 25.4 25.4) (xy 22.86 25.4))
+      (at 17.78 101.6 0)
+      (effects (font (size 1.27 1.27)))
+    )
+    (pin "1")
+  )
+  (wire
+    (pts (xy 20.32 99.06) (xy 17.78 99.06))
+    (stroke (width 0) (type default))
+  )
+  (wire
+    (pts (xy 20.32 96.52) (xy 17.78 96.52))
     (stroke (width 0) (type default))
   )
   (symbol
     (lib_id "74xx:74AHC1G14")
-    (at 190.5 30.48 0)
+    (at 63.5 368.3 0)
     (unit 1)
     (exclude_from_sim no)
@@
     (dnp no)
     (property "Reference" "U2"
-      (at 193.04 27.94 0)
+      (at 66.04 365.76 0)
       (effects (font (size 1.27 1.27)))
     )
     (property "Value" "SN74AHC1G14"
-      (at 190.5 33.02 0)
+      (at 63.5 370.84 0)
       (effects (font (size 1.27 1.27)))
     )
@@
   (symbol
     (lib_id "Device:D_Zener")
-    (at 30.48 69.85 0)
+    (at 63.5 25.4 0)
     (unit 1)
     (exclude_from_sim no)
@@
     (dnp no)
     (property "Reference" "D1"
-      (at 33.02 67.31 0)
+      (at 66.04 22.86 0)
       (effects (font (size 1.27 1.27)))
     )
     (property "Value" "1N4728A"
-      (at 30.48 72.39 0)
-      (effects (font (size 1.27 1.27)))
-    )
-    (pin "1")
-    (pin "2")
-  )
-  (wire
-    (pts (xy 26.67 69.85) (xy 24.13 69.85))
-    (stroke (width 0) (type default))
-  )
-  (wire
-    (pts (xy 34.29 69.85) (xy 36.83 69.85))
+      (at 63.5 27.94 0)
+      (effects (font (size 1.27 1.27)))
+    )
+    (pin "1")
+    (pin "2")
+  )
+  (wire
+    (pts (xy 59.69 25.4) (xy 57.15 25.4))
+    (stroke (width 0) (type default))
+  )
+  (wire
+    (pts (xy 67.31 25.4) (xy 69.85 25.4))
     (stroke (width 0) (type default))
   )
   (symbol
     (lib_id "Device:R")
-    (at 69.85 69.85 0)
+    (at 63.5 215.9 0)
     (unit 1)
     (exclude_from_sim no)
@@
     (dnp no)
     (property "Reference" "R1"
-      (at 72.39 67.31 0)
+      (at 66.04 213.36 0)
       (effects (font (size 1.27 1.27)))
     )
     (property "Value" "1e+04 Ω"
-      (at 69.85 72.39 0)
-      (effects (font (size 1.27 1.27)))
-    )
-    (pin "1")
-    (pin "2")
-  )
-  (wire
-    (pts (xy 69.85 73.66) (xy 69.85 76.2))
-    (stroke (width 0) (type default))
-  )
-  (wire
-    (pts (xy 69.85 66.04) (xy 69.85 63.5))
+      (at 63.5 218.44 0)
+      (effects (font (size 1.27 1.27)))
+    )
+    (pin "1")
+    (pin "2")
+  )
+  (wire
+    (pts (xy 63.5 219.71) (xy 63.5 222.25))
+    (stroke (width 0) (type default))
+  )
+  (wire
+    (pts (xy 63.5 212.09) (xy 63.5 209.55))
     (stroke (width 0) (type default))
   )
   (symbol
     (lib_id "Device:R")
-    (at 110.49 69.85 0)
+    (at 63.5 254 0)
     (unit 1)
     (exclude_from_sim no)
@@
     (dnp no)
     (property "Reference" "R2"
-      (at 113.03 67.31 0)
+      (at 66.04 251.46 0)
       (effects (font (size 1.27 1.27)))
     )
     (property "Value" "1e+04 Ω"
-      (at 110.49 72.39 0)
-      (effects (font (size 1.27 1.27)))
-    )
-    (pin "1")
-    (pin "2")
-  )
-  (wire
-    (pts (xy 110.49 73.66) (xy 110.49 76.2))
-    (stroke (width 0) (type default))
-  )
-  (wire
-    (pts (xy 110.49 66.04) (xy 110.49 63.5))
+      (at 63.5 256.54 0)
+      (effects (font (size 1.27 1.27)))
+    )
+    (pin "1")
+    (pin "2")
+  )
+  (wire
+    (pts (xy 63.5 257.81) (xy 63.5 260.35))
+    (stroke (width 0) (type default))
+  )
+  (wire
+    (pts (xy 63.5 250.19) (xy 63.5 247.65))
     (stroke (width 0) (type default))
   )
   (symbol
     (lib_id "Device:R")
-    (at 149.86 69.85 0)
+    (at 63.5 292.1 0)
     (unit 1)
     (exclude_from_sim no)
@@
     (dnp no)
     (property "Reference" "R3"
-      (at 152.4 67.31 0)
+      (at 66.04 289.56 0)
       (effects (font (size 1.27 1.27)))
     )
     (property "Value" "1e+04 Ω"
-      (at 149.86 72.39 0)
-      (effects (font (size 1.27 1.27)))
-    )
-    (pin "1")
-    (pin "2")
-  )
-  (wire
-    (pts (xy 149.86 73.66) (xy 149.86 76.2))
-    (stroke (width 0) (type default))
-  )
-  (wire
-    (pts (xy 149.86 66.04) (xy 149.86 63.5))
+      (at 63.5 294.64 0)
+      (effects (font (size 1.27 1.27)))
+    )
+    (pin "1")
+    (pin "2")
+  )
+  (wire
+    (pts (xy 63.5 295.91) (xy 63.5 298.45))
+    (stroke (width 0) (type default))
+  )
+  (wire
+    (pts (xy 63.5 288.29) (xy 63.5 285.75))
     (stroke (width 0) (type default))
   )
   (symbol
     (lib_id "Connector_Generic:Conn_01x04")
-    (at 190.5 69.85 0)
+    (at 25.4 25.4 0)
     (unit 1)
     (exclude_from_sim no)
@@
     (dnp no)
     (property "Reference" "J1"
-      (at 193.04 67.31 0)
+      (at 27.94 22.86 0)
       (effects (font (size 1.27 1.27)))
     )
     (property "Value" "Header1xNFemale"
-      (at 190.5 72.39 0)
+      (at 25.4 27.94 0)
       (effects (font (size 1.27 1.27)))
     )
@@
   )
   (wire
-    (pts (xy 185.42 72.39) (xy 182.88 72.39))
+    (pts (xy 20.32 27.94) (xy 17.78 27.94))
     (stroke (width 0) (type default))
   )
   (symbol
     (lib_id "power:VCC")
-    (at 182.88 72.39 90)
+    (at 17.78 27.94 90)
     (unit 1)
     (exclude_from_sim no)
@@
     (dnp no)
     (property "Reference" "#PWR"
-      (at 182.88 72.39 0)
+      (at 17.78 27.94 0)
       (effects (font (size 1.27 1.27)) (hide yes))
     )
     (property "Value" "VCC"
-      (at 182.88 72.39 0)
-      (effects (font (size 1.27 1.27)))
-    )
-    (pin "1")
-  )
-  (wire
-    (pts (xy 185.42 69.85) (xy 182.88 69.85))
+      (at 17.78 27.94 0)
+      (effects (font (size 1.27 1.27)))
+    )
+    (pin "1")
+  )
+  (wire
+    (pts (xy 20.32 25.4) (xy 17.78 25.4))
     (stroke (width 0) (type default))
   )
   (symbol
     (lib_id "power:GND")
-    (at 182.88 69.85 270)
+    (at 17.78 25.4 270)
     (unit 1)
     (exclude_from_sim no)
@@
     (dnp no)
     (property "Reference" "#PWR"
-      (at 182.88 69.85 0)
+      (at 17.78 25.4 0)
       (effects (font (size 1.27 1.27)) (hide yes))
     )
     (property "Value" "GND"
-      (at 182.88 69.85 0)
-      (effects (font (size 1.27 1.27)))
-    )
-    (pin "1")
-  )
-  (wire
-    (pts (xy 185.42 67.31) (xy 182.88 67.31))
-    (stroke (width 0) (type default))
-  )
-  (wire
-    (pts (xy 185.42 64.77) (xy 182.88 64.77))
+      (at 17.78 25.4 0)
+      (effects (font (size 1.27 1.27)))
+    )
+    (pin "1")
+  )
+  (wire
+    (pts (xy 20.32 22.86) (xy 17.78 22.86))
+    (stroke (width 0) (type default))
+  )
+  (wire
+    (pts (xy 20.32 20.32) (xy 17.78 20.32))
     (stroke (width 0) (type default))
   )
   (symbol
     (lib_id "Connector_Generic:Conn_01x04")
-    (at 229.87 69.85 0)
+    (at 25.4 63.5 0)
     (unit 1)
     (exclude_from_sim no)
@@
     (dnp no)
     (property "Reference" "J2"
-      (at 232.41 67.31 0)
+      (at 27.94 60.96 0)
       (effects (font (size 1.27 1.27)))
     )
     (property "Value" "Header1xNFemale"
-      (at 229.87 72.39 0)
+      (at 25.4 66.04 0)
       (effects (font (size 1.27 1.27)))
     )
@@
   )
   (wire
-    (pts (xy 224.79 72.39) (xy 222.25 72.39))
-    (stroke (width 0) (type default))
-  )
-  (wire
-    (pts (xy 224.79 69.85) (xy 222.25 69.85))
-    (stroke (width 0) (type default))
-  )
-  (wire
-    (pts (xy 224.79 67.31) (xy 222.25 67.31))
-    (stroke (width 0) (type default))
-  )
-  (wire
-    (pts (xy 224.79 64.77) (xy 222.25 64.77))
-    (stroke (width 0) (type default))
-  )
+    (pts (xy 20.32 66.04) (xy 17.78 66.04))
+    (stroke (width 0) (type default))
+  )
+  (wire
+    (pts (xy 20.32 63.5) (xy 17.78 63.5))
+    (stroke (width 0) (type default))
+  )
+  (wire
+    (pts (xy 20.32 60.96) (xy 17.78 60.96))
+    (stroke (width 0) (type default))
+  )
+  (wire
+    (pts (xy 20.32 58.42) (xy 17.78 58.42))
+    (stroke (width 0) (type default))
+  )

Commit message: export: kicad_sch — Phase 2.5c: hierarchical sheets for multi-Board designs
Multi-Board assembly designs (WaterAlarmAssembly, BLDCSystem,
IsolatedRS232Link, CooledSystem) previously emitted a single giant
flat schematic (88.9 mm × 660–700 mm) by dumping all boards' parts
into one layout.  Phase 2.5c replaces this with proper KiCad
hierarchical schematics:

  - <Design>.kicad_sch — top-level system sheet with one (sheet ...)
    block per Board, sized A4/A3 instead of the previous strip.
  - <Design>__<BoardClass>.kicad_sch — flat Board sub-sheet (one per Board).

render_all(design, ctx) -> dict[str, str] is the new multi-file
entry point; export_to_string / render() also return the top-level
sheet for multi-Board designs (was: flat dump, effectively unusable).

scripts/render_demo_docs.py updated to call render_all and write
all returned files (top-level + sub-sheets) into the demo's docs/.

13 new tests in test_hierarchical.py; 69 kicad_sch tests total.
Parts:
- removed D1: 1N4728A, symbol Device:D_Zener
- removed J1, J2: Header1xNFemale, symbol Connector_Generic:Conn_01x04
- removed P1: Header1xNMale, symbol Connector_Generic:Conn_01x04
- removed R1, R2, R3: 1e+04 Ω, symbol Device:R
- removed U2: SN74AHC1G14, symbol 74xx:74AHC1G14
Other:
- added sheet FanCoolingBoard (CooledSystem__FanCoolingBoard.kicad_sch)
- added sheet PowerSourceBoard (CooledSystem__PowerSourceBoard.kicad_sch)
