File: demos/fan_cooling/docs/CooledSystem__FanCoolingBoard.kicad_sch (KiCad schematic)
At the start: 7 parts, among them J1 Header1xNFemale, J2 Header1xNFemale, U2 SN74AHC1G14

Commit message: framework: passive + diode terminals mandatory (#30)
Continuation of the LED.cathode regression fix (#29). Resistor,
Capacitor, Inductor, and every Diode subclass had their terminals
declared `mandatory=False` with the same "structurally inert under
graph evaluation" justification — letting demos declare BOM-only
timing / decoupling / pull-up parts without wiring them, then ship
breadboard SVGs and netlists where those parts sat orphaned.

A real resistor / capacitor / inductor / diode with a dangling
terminal does nothing. Marking the ports mandatory closes the
silent regression at the framework layer.

  - `src/components/passives/{resistor,capacitor,inductor}.py` and
    every diode subclass under `src/components/diodes/` now declare
    their terminals `mandatory=True`.
  - `tests/components/test_{resistor,capacitor,inductor}.py`:
    regression tests pin the new contract per component.
  - `tests/components/test_diode_mandatory_terminals.py` (new):
    parametrized over D1N4001 / D1N4007 / D1N4148 / D1N4728A /
    D1N4733A / D1N4742A / D1N5817.
  - Six demos (`backup_power`, `bldc_motor`, `dice`,
    `doorbell_protector`, `fan_cooling`, `isolated_rs232`) had
    declared-but-unwired passives — each now wires them either to
    their datasheet-correct net (e.g. DoorbellProtector's flyback
    diode anode joins the relay coil_minus net) or as an isolated
    0-Ω passthrough with `dynamically_driven=True` where the part
    is genuinely BOM-only and the voltage-only simulator can't
    honour its behaviour. Comments at each call site explain
    which kind.
  - Test fixtures across CLI, refdes, format-roundtrip, kicad
    import, and per-format renderer tests updated so they still
    pin down the specific error each one exists to catch without
    tripping the new mandatory-pin check first.
  - All demo docs regenerated; goldens refreshed.

After this commit the breadboard SVGs show every BOM part connected
to something — no more orphaned caps and resistors float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
Connections:
- net Net-(D1-anode): now reaches D1.1 (K)
- net Net-(D1-anode): now also D1.2 (A)
- net Net-(R3-t1): now reaches R3.1
- net Net-(R3-t1): now also R3.2
- net Net-(R2-t1): now reaches R2.1
- net Net-(R2-t1): now also R2.2
- net Net-(R1-t1): now reaches R1.1
- net Net-(R1-t1): now also R1.2
Changed lines of the file:
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@@
     (stroke (width 0) (type default))
+  )
+  (global_label "Net-(D1-anode)"
+    (shape input)
+    (at 57.15 25.4 0)
+    (fields_autoplaced yes)
+    (effects (font (size 1.27 1.27)) (justify right))
+    (property "Intersheet References" "${INTERSHEET_REFS}"
+      (at 0 0 0)
+      (effects (font (size 1.27 1.27)) (hide yes))
+    )
   )
   (wire
     (pts (xy 67.31 25.4) (xy 69.85 25.4))
     (stroke (width 0) (type default))
+  )
+  (global_label "Net-(D1-anode)"
+    (shape input)
+    (at 69.85 25.4 0)
+    (fields_autoplaced yes)
+    (effects (font (size 1.27 1.27)) (justify right))
+    (property "Intersheet References" "${INTERSHEET_REFS}"
+      (at 0 0 0)
+      (effects (font (size 1.27 1.27)) (hide yes))
+    )
   )
   (symbol
@@
     (stroke (width 0) (type default))
   )
+  (global_label "Net-(R1-t1)"
+    (shape input)
+    (at 63.5 222.25 0)
+    (fields_autoplaced yes)
+    (effects (font (size 1.27 1.27)) (justify right))
+    (property "Intersheet References" "${INTERSHEET_REFS}"
+      (at 0 0 0)
+      (effects (font (size 1.27 1.27)) (hide yes))
+    )
+  )
   (wire
     (pts (xy 63.5 212.09) (xy 63.5 209.55))
     (stroke (width 0) (type default))
+  )
+  (global_label "Net-(R1-t1)"
+    (shape input)
+    (at 63.5 209.55 0)
+    (fields_autoplaced yes)
+    (effects (font (size 1.27 1.27)) (justify right))
+    (property "Intersheet References" "${INTERSHEET_REFS}"
+      (at 0 0 0)
+      (effects (font (size 1.27 1.27)) (hide yes))
+    )
   )
   (symbol
@@
     (stroke (width 0) (type default))
   )
+  (global_label "Net-(R2-t1)"
+    (shape input)
+    (at 63.5 260.35 0)
+    (fields_autoplaced yes)
+    (effects (font (size 1.27 1.27)) (justify right))
+    (property "Intersheet References" "${INTERSHEET_REFS}"
+      (at 0 0 0)
+      (effects (font (size 1.27 1.27)) (hide yes))
+    )
+  )
   (wire
     (pts (xy 63.5 250.19) (xy 63.5 247.65))
     (stroke (width 0) (type default))
+  )
+  (global_label "Net-(R2-t1)"
+    (shape input)
+    (at 63.5 247.65 0)
+    (fields_autoplaced yes)
+    (effects (font (size 1.27 1.27)) (justify right))
+    (property "Intersheet References" "${INTERSHEET_REFS}"
+      (at 0 0 0)
+      (effects (font (size 1.27 1.27)) (hide yes))
+    )
   )
   (symbol
@@
     (stroke (width 0) (type default))
   )
+  (global_label "Net-(R3-t1)"
+    (shape input)
+    (at 63.5 298.45 0)
+    (fields_autoplaced yes)
+    (effects (font (size 1.27 1.27)) (justify right))
+    (property "Intersheet References" "${INTERSHEET_REFS}"
+      (at 0 0 0)
+      (effects (font (size 1.27 1.27)) (hide yes))
+    )
+  )
   (wire
     (pts (xy 63.5 288.29) (xy 63.5 285.75))
     (stroke (width 0) (type default))
+  )
+  (global_label "Net-(R3-t1)"
+    (shape input)
+    (at 63.5 285.75 0)
+    (fields_autoplaced yes)
+    (effects (font (size 1.27 1.27)) (justify right))
+    (property "Intersheet References" "${INTERSHEET_REFS}"
+      (at 0 0 0)
+      (effects (font (size 1.27 1.27)) (hide yes))
+    )
   )
   (symbol
@@
     (stroke (width 0) (type default))
   )
+  (wire
+    (pts (xy 57.15 25.4) (xy 69.85 25.4))
+    (stroke (width 0) (type default))
+  )
+  (wire
+    (pts (xy 63.5 209.55) (xy 63.5 222.25))
+    (stroke (width 0) (type default))
+  )
+  (wire
+    (pts (xy 63.5 247.65) (xy 63.5 260.35))
+    (stroke (width 0) (type default))
+  )
+  (wire
+    (pts (xy 63.5 285.75) (xy 63.5 298.45))
+    (stroke (width 0) (type default))
+  )

Commit message: units: Ohms.__str__ uses engineering notation (kΩ, MΩ, GΩ)
The previous `Ohms.__str__` formatted with bare `:.3g`, producing
unreadable scientific output for clean kilo / mega multiples:

  str(Ohms(10_000))     == "1e+04 Ω"      → now "10 kΩ"
  str(Ohms(100_000))    == "1e+05 Ω"      → now "100 kΩ"
  str(Ohms(1_000_000))  == "1e+06 Ω"      → now "1 MΩ"

The breadboard SVG visualiser surfaced the problem: a resistor body
labelled "100000Ω" makes a reader count zeros, while a label of
"100 kΩ" reads at a glance — exactly the convention every schematic
and parts catalogue uses. Centralising the engineering notation in
`Ohms.__str__` means every downstream consumer (assembly guide,
breadboard SVG, kicad netlist, BOM, reports) inherits the readable
form without each format adapter rolling its own formatter.

  - `Ohms.__str__` returns "47 Ω", "4.7 kΩ", "10 kΩ", "100 kΩ",
    "1 MΩ", "10 MΩ", "1 GΩ" per the kilo / mega / giga thresholds.
  - `Resistor.__str__` delegates to `str(self._ohms)` so it
    inherits the new notation (was producing the noisy "47.0 Ω"
    via raw float).
  - The breadboard visualiser's resistor body label uses
    `str(part.ohms)` directly (previously had a private
    `_format_ohms_compact` helper; removed).
  - `tests/components/test_resistor.py::test_str` updated for
    "47 Ω" (was "47.0 Ω"); new `test_str_renders_in_engineering_notation`
    pins kΩ / MΩ output across the kilo and mega thresholds.
  - All demo docs / goldens refreshed where the Ohms.__str__
    change affected the rendered output (breadboard SVGs, kicad
    sch value fields, BOM rows).
Parts:
- R1, R2, R3: value 1e+04 Ω -> 10 kΩ
Changed lines of the file:
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@@
       (effects (font (size 1.27 1.27)))
     )
-    (property "Value" "1e+04 Ω"
+    (property "Value" "10 kΩ"
       (at 63.5 218.44 0)
       (effects (font (size 1.27 1.27)))
@@
       (effects (font (size 1.27 1.27)))
     )
-    (property "Value" "1e+04 Ω"
+    (property "Value" "10 kΩ"
       (at 63.5 256.54 0)
       (effects (font (size 1.27 1.27)))
@@
       (effects (font (size 1.27 1.27)))
     )
-    (property "Value" "1e+04 Ω"
+    (property "Value" "10 kΩ"
       (at 63.5 294.64 0)
       (effects (font (size 1.27 1.27)))
