File: demos/water_alarm_split/docs/WaterAlarmAssembly__ControllerBoard.kicad_sch (KiCad schematic)
At the start: 4 parts, among them U1 SN74HC04, U2 CD4069

Commit message: framework: LED.cathode mandatory + close WaterAlarm regression (#29)
Found while reviewing WaterAlarm's breadboard SVG: the LEDs in the
design had no ground connections drawn. Investigation revealed
`LED.cathode` was declared `mandatory=False` with the docstring claim
*"floating = GND"* — a "structurally inert under graph evaluation"
shortcut that lets demos write electrically-broken circuits and have
them pass ERC.

A real LED with a dangling cathode does not light. This is exactly
the kind of physical-fidelity violation `CLAUDE.md` lists as
disallowed.

  - `src/components/passives/led.py`: `cathode` becomes
    `mandatory=True`. Docstring updated to drop the "floating = GND"
    claim and explain the contract.
  - `tests/components/test_led.py`: regression tests pin both ports
    as mandatory and confirm `Circuit.__init__` raises
    `UnconnectedPinError` end-to-end when a cathode is left
    floating.
  - `demos/water_alarm/water_alarm.py` and
    `demos/water_alarm_split/water_alarm_split.py`: cathodes wired
    to the GND rail. (Bench builds still need a series current-limit
    resistor; the logic-level demo doesn't model V_F or current.)
  - `tests/framework/test_circuit_autocollect.py`,
    `tests/framework/test_framework.py`, and
    `tests/framework/import_kicad/test_import.py`: fixtures that
    leaned on the broken default updated so they still pin down the
    specific error each test exists to catch.
  - Demo docs regenerated for the two WaterAlarm variants.
Connections:
- net Net-(D2-anode) is gone; now on net GND: D2.1 (K), D2.2 (A), U2.2
- net GND: now also D1.2 (A)
Changed lines of the file:
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@@
+  )
+  (symbol
+    (lib_id "power:GND")
+    (at 69.85 927.1 270)
+    (unit 1)
+    (exclude_from_sim no)
+    (in_bom yes)
+    (on_board yes)
+    (dnp no)
+    (property "Reference" "#PWR"
+      (at 69.85 927.1 0)
+      (effects (font (size 1.27 1.27)) (hide yes))
+    )
+    (property "Value" "GND"
+      (at 69.85 927.1 0)
+      (effects (font (size 1.27 1.27)))
+    )
+    (pin "1")
   )
   (symbol
@@
     (stroke (width 0) (type default))
   )
+  (symbol
+    (lib_id "power:GND")
+    (at 69.85 965.2 270)
+    (unit 1)
+    (exclude_from_sim no)
+    (in_bom yes)
+    (on_board yes)
+    (dnp no)
+    (property "Reference" "#PWR"
+      (at 69.85 965.2 0)
+      (effects (font (size 1.27 1.27)) (hide yes))
+    )
+    (property "Value" "GND"
+      (at 69.85 965.2 0)
+      (effects (font (size 1.27 1.27)))
+    )
+    (pin "1")
+  )
   (wire
