File: demos/backup_power/docs/BackupPower.kicad_sch (KiCad schematic)
At the start: 21 parts, among them U2 LM5002

Commit message: export: kicad_sch — Phase 2.5b: layered placement, wire routing, KiCad 10 compatibility (#23)
* export: kicad_sch — Phase 2.5b: layered placement + routing + KiCad 9 fix

Placement (placement.py, complete rewrite):
- Replaces naive grid with Layered Signal Flow algorithm (spec §5 stages 1–8)
- Stage 1: band classification — power chips/rails at top, LEDs at bottom,
  everything else in the signal band
- Stage 2: signal-flow DAG via BFS from Rail/Connector sources; layer = BFS
  distance from nearest source
- Stage 3–4: place within (band, layer) cells at 1500-mil (38.1 mm) same-band
  spacing, 1000-mil inter-band gutter, 25.4 mm page margin
- Stage 6: cluster breakup — up to 10 iterations shifting same-band parts
  that land closer than 0.9× SAME_BAND_SPACING_MM
- Stage 8: page sized to fit (A4 → A3 → A2 → A1)
- grid_place() and sheet_size_mm() kept as shims for backward-compat

Routing (routing.py, new file):
- route_net(): connects stub ends with Manhattan L-shapes (horizontal first)
- find_junctions(): returns points where ≥3 wire endpoints coincide
- renderer uses routed wires between signal-net stub ends

Hierarchical (hierarchical.py, new file):
- collect_boards(), is_multi_board(), sub_sheet_filename() — interface stub
  for multi-Board sub-sheet emission (full implementation deferred)

KiCad 9 sub-symbol name fix (library_loader.py):
- KiCad 9 schematics expect sub-symbols nested inside their parent in
  lib_symbols to use the bare name (R_0_1, LED_0_1, 4069_1_0) — NOT the
  lib-qualified name (Device:R_0_1, Device:LED_0_1, 4xxx:4069_1_0)
- Fixed _qualify_names() to add the lib: prefix only to the exact parent
  symbol name using a lookahead (?=") that prevents sub-unit names from
  being qualified

Tests (+25 tests):
- test_placement.py: band classification, all-on-grid, determinism,
  minimum spacing, power < signal < indicator Y ordering, page sizing
- test_routing.py: H/V segments, L-shapes, orthogonality, grid snap,
  junction detection

Golden files re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
Other:
- moved on the sheet: C1, C10, C12, C13, C14, C15, C2, C3, C4, C5, C6, C7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

Commit message: framework: passive + diode terminals mandatory (#30)
Continuation of the LED.cathode regression fix (#29). Resistor,
Capacitor, Inductor, and every Diode subclass had their terminals
declared `mandatory=False` with the same "structurally inert under
graph evaluation" justification — letting demos declare BOM-only
timing / decoupling / pull-up parts without wiring them, then ship
breadboard SVGs and netlists where those parts sat orphaned.

A real resistor / capacitor / inductor / diode with a dangling
terminal does nothing. Marking the ports mandatory closes the
silent regression at the framework layer.

  - `src/components/passives/{resistor,capacitor,inductor}.py` and
    every diode subclass under `src/components/diodes/` now declare
    their terminals `mandatory=True`.
  - `tests/components/test_{resistor,capacitor,inductor}.py`:
    regression tests pin the new contract per component.
  - `tests/components/test_diode_mandatory_terminals.py` (new):
    parametrized over D1N4001 / D1N4007 / D1N4148 / D1N4728A /
    D1N4733A / D1N4742A / D1N5817.
  - Six demos (`backup_power`, `bldc_motor`, `dice`,
    `doorbell_protector`, `fan_cooling`, `isolated_rs232`) had
    declared-but-unwired passives — each now wires them either to
    their datasheet-correct net (e.g. DoorbellProtector's flyback
    diode anode joins the relay coil_minus net) or as an isolated
    0-Ω passthrough with `dynamically_driven=True` where the part
    is genuinely BOM-only and the voltage-only simulator can't
    honour its behaviour. Comments at each call site explain
    which kind.
  - Test fixtures across CLI, refdes, format-roundtrip, kicad
    import, and per-format renderer tests updated so they still
    pin down the specific error each one exists to catch without
    tripping the new mandatory-pin check first.
  - All demo docs regenerated; goldens refreshed.

After this commit the breadboard SVGs show every BOM part connected
to something — no more orphaned caps and resistors float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
Connections:
- net VCC: now reaches C14.1
- net VCC: now also C1.1, C1.2, C10.1, C10.2, C12.1, C12.2, C13.1, C13.2, C14.2, C15.1, C15.2, C2.1, C2.2, C3.1, C3.2, C4.1, C4.2, C5.1, C5.2, C6.1, C6.2, C7.1, C7.2, C8.1, C8.2, C9.1, C9.2, L1.1, L1.2, R11.1, R11.2, R16.1, R16.2, R6.1, R6.2, R7.1, R7.2

Commit message: units: Ohms.__str__ uses engineering notation (kΩ, MΩ, GΩ) (#33)
* units: Ohms.__str__ uses engineering notation (kΩ, MΩ, GΩ)

The previous `Ohms.__str__` formatted with bare `:.3g`, producing
unreadable scientific output for clean kilo / mega multiples:

  str(Ohms(10_000))     == "1e+04 Ω"      → now "10 kΩ"
  str(Ohms(100_000))    == "1e+05 Ω"      → now "100 kΩ"
  str(Ohms(1_000_000))  == "1e+06 Ω"      → now "1 MΩ"

The breadboard SVG visualiser surfaced the problem: a resistor body
labelled "100000Ω" makes a reader count zeros, while a label of
"100 kΩ" reads at a glance — exactly the convention every schematic
and parts catalogue uses. Centralising the engineering notation in
`Ohms.__str__` means every downstream consumer (assembly guide,
breadboard SVG, kicad netlist, BOM, reports) inherits the readable
form without each format adapter rolling its own formatter.

  - `Ohms.__str__` returns "47 Ω", "4.7 kΩ", "10 kΩ", "100 kΩ",
    "1 MΩ", "10 MΩ", "1 GΩ" per the kilo / mega / giga thresholds.
  - `Resistor.__str__` delegates to `str(self._ohms)` so it
    inherits the new notation (was producing the noisy "47.0 Ω"
    via raw float).
  - The breadboard visualiser's resistor body label uses
    `str(part.ohms)` directly (previously had a private
    `_format_ohms_compact` helper; removed).
  - `tests/components/test_resistor.py::test_str` updated for
    "47 Ω" (was "47.0 Ω"); new `test_str_renders_in_engineering_notation`
    pins kΩ / MΩ output across the kilo and mega thresholds.
  - All demo docs / goldens refreshed where the Ohms.__str__
    change affected the rendered output (breadboard SVGs, kicad
    sch value fields, BOM rows).

* units: Farads + Henries __str__ also use engineering notation

Same treatment as `Ohms.__str__` (previous commit) for the other two
passive engineering quantities. Demos contain caps and inductors
with values that the bare `:.3g` formatter would emit in scientific
form (`1e-07 F` for a 100 nF decoupling cap); centralising t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
Parts:
- C1: value 1e-08 F -> 10 nF
- C10: value 0.0012 F -> 1.2 mF
- C12, C14, C2, C3, C6, C8: value 1e-06 F -> 1 µF
- C13: value 0.00022 F -> 220 µF
- C15: value 2.2e-06 F -> 2.2 µF
- C4: value 3.3e-09 F -> 3.3 nF
- C5: value 2.2e-08 F -> 22 nF
- C7, C9: value 1e-07 F -> 100 nF
- L1: value 3.3e-05 H -> 33 µH
- R11: value 4.02e+04 Ω -> 40.2 kΩ
- R16: value 1e+04 Ω -> 10 kΩ
- R6: value 7.15e+05 Ω -> 715 kΩ
- R7: value 2.26e+05 Ω -> 226 kΩ
Changed lines of the file:
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@@
       (effects (font (size 1.27 1.27)))
     )
-    (property "Value" "3.3e-05 H"
+    (property "Value" "33 µH"
       (at 63.5 929.64 0)
       (effects (font (size 1.27 1.27)))
@@
       (effects (font (size 1.27 1.27)))
     )
-    (property "Value" "0.0012 F"
+    (property "Value" "1.2 mF"
       (at 63.5 472.44 0)
       (effects (font (size 1.27 1.27)))
@@
       (effects (font (size 1.27 1.27)))
     )
-    (property "Value" "1e-08 F"
+    (property "Value" "10 nF"
       (at 63.5 129.54 0)
       (effects (font (size 1.27 1.27)))
@@
       (effects (font (size 1.27 1.27)))
     )
-    (property "Value" "1e-06 F"
+    (property "Value" "1 µF"
       (at 63.5 167.64 0)
       (effects (font (size 1.27 1.27)))
@@
       (effects (font (size 1.27 1.27)))
     )
-    (property "Value" "1e-06 F"
+    (property "Value" "1 µF"
       (at 63.5 205.74 0)
       (effects (font (size 1.27 1.27)))
@@
       (effects (font (size 1.27 1.27)))
     )
-    (property "Value" "3.3e-09 F"
+    (property "Value" "3.3 nF"
       (at 63.5 243.84 0)
       (effects (font (size 1.27 1.27)))
@@
       (effects (font (size 1.27 1.27)))
     )
-    (property "Value" "2.2e-08 F"
+    (property "Value" "22 nF"
       (at 63.5 281.94 0)
       (effects (font (size 1.27 1.27)))
@@
       (effects (font (size 1.27 1.27)))
     )
-    (property "Value" "1e-06 F"
+    (property "Value" "1 µF"
       (at 63.5 320.04 0)
       (effects (font (size 1.27 1.27)))
@@
       (effects (font (size 1.27 1.27)))
     )
-    (property "Value" "1e-07 F"
+    (property "Value" "100 nF"
       (at 63.5 358.14 0)
       (effects (font (size 1.27 1.27)))
@@
       (effects (font (size 1.27 1.27)))
     )
-    (property "Value" "1e-06 F"
+    (property "Value" "1 µF"
       (at 63.5 396.24 0)
       (effects (font (size 1.27 1.27)))
@@
       (effects (font (size 1.27 1.27)))
     )
-    (property "Value" "1e-07 F"
+    (property "Value" "100 nF"
       (at 63.5 434.34 0)
       (effects (font (size 1.27 1.27)))
@@
       (effects (font (size 1.27 1.27)))
     )
-    (property "Value" "1e-06 F"
+    (property "Value" "1 µF"
       (at 63.5 510.54 0)
       (effects (font (size 1.27 1.27)))
@@
       (effects (font (size 1.27 1.27)))
     )
-    (property "Value" "0.00022 F"
+    (property "Value" "220 µF"
       (at 63.5 548.64 0)
       (effects (font (size 1.27 1.27)))
@@
       (effects (font (size 1.27 1.27)))
     )
-    (property "Value" "1e-06 F"
+    (property "Value" "1 µF"
       (at 63.5 586.74 0)
       (effects (font (size 1.27 1.27)))
@@
       (effects (font (size 1.27 1.27)))
     )
-    (property "Value" "2.2e-06 F"
+    (property "Value" "2.2 µF"
       (at 63.5 624.84 0)
       (effects (font (size 1.27 1.27)))
@@
       (effects (font (size 1.27 1.27)))
     )
-    (property "Value" "7.15e+05 Ω"
+    (property "Value" "715 kΩ"
       (at 63.5 967.74 0)
       (effects (font (size 1.27 1.27)))
@@
       (effects (font (size 1.27 1.27)))
     )
-    (property "Value" "2.26e+05 Ω"
+    (property "Value" "226 kΩ"
       (at 63.5 1005.84 0)
       (effects (font (size 1.27 1.27)))
@@
       (effects (font (size 1.27 1.27)))
     )
-    (property "Value" "4.02e+04 Ω"
+    (property "Value" "40.2 kΩ"
       (at 63.5 1043.94 0)
       (effects (font (size 1.27 1.27)))
@@
       (effects (font (size 1.27 1.27)))
     )
-    (property "Value" "1e+04 Ω"
+    (property "Value" "10 kΩ"
       (at 63.5 1082.04 0)
       (effects (font (size 1.27 1.27)))
